Commit message: Camera Rearranged

File: src/robot_description/model/robot.xacro (robot description, xacro)
@@ -151,5 +151,5 @@
     <!-- Position above the body (z offset = body height / 2 + 0.05) -->
     <child link="camera_link"/>
-    <origin xyz="0 0 0.6" rpy="0 0 0"/>
+    <origin xyz="0.5 0 0.3" rpy="0 0 0"/>
     <axis xyz="0 0 1"/>
   </joint>

Commit message: Added_lidar and  new World

File: src/robot_description/model/robot.xacro (robot description, xacro)
@@ -170,3 +170,27 @@
     </collision>
   </link>
+    <!-- lidar -->
+  <joint name="lidar_joint" type="fixed">
+    <parent link="body_link"/>
+    <!-- Position above the body (z offset = body height / 2 + 0.05) -->
+    <child link="lidar_link"/>
+    <origin xyz="0 0 0.47" rpy="0 0 0"/>
+    <axis xyz="0 0 1"/>
+  </joint>
+  <link name="lidar_link">
+    <inertial>
+      <mass value="0.1"/>
+      <inertia ixx="0.000416667" ixy="0" ixz="0" iyy="0.000416667" iyz="0" izz="0.0008"/>
+    </inertial>
+    <visual name="visual">
+      <geometry>
+        <cylinder radius="0.1" length="0.05"/>
+      </geometry>
+    </visual>
+    <collision name="collision">
+      <geometry>
+        <cylinder radius="0.04" length="0.05"/>
+      </geometry>
+    </collision>
+  </link>
 </robot>
